Commit message: update

File: arm_controller/chains/arm.urdf (robot description, URDF)
Before this commit: robot MechaArm, 8 links, 7 joints
Joints:
- joint base: origin xyz=0 0 56.0 rpy=0 0 1.57 -> xyz=0 0 56.0 rpy=0 0 0
- joint waist: origin xyz=0 0 42.93 rpy=0 0 0 -> xyz=0 0 42.93 rpy=0 0 1.57

Commit message: visualized arm, added rpy

File: arm_controller/chains/arm.urdf (robot description, URDF)
Before this commit: robot MechaArm, 8 links, 7 joints
Links:
- added link claw_left_link; visual box size=0.02 0.02 0.06
- added link claw_right_link; visual box size=0.02 0.02 0.06
- link base_waist_link: geometry visual cylinder length=0.01 radius=0.035
- link claw_end_link: geometry visual box size=0.01 0.03 0.03
- link elbow_wrist_roll_link: geometry visual box size=0.030 0.015 0.06
- link shoulder_elbow_link: geometry visual box size=0.030 0.015 0.120
- link waist_shoulder_link: geometry visual cylinder length=0.02 radius=0.015
- link world_base_link: geometry visual cylinder length=0.056 radius=0.04
- link wrist_pitch_claw_link: geometry visual box size=0.03 0.03 0.03
- link wrist_roll_wrist_pitch_link: geometry visual box size=0.024 0.012 0.03
Joints:
- added joint claw_left: type fixed, parent wrist_pitch_claw_link, child claw_left_link, origin xyz=0 .015 0 rpy=0 0 0
- added joint claw_right: type fixed, parent wrist_pitch_claw_link, child claw_right_link, origin xyz=0 -.015 0 rpy=0 0 0
- joint base: origin xyz=0 0 56.0 rpy=0 0 0 -> xyz=0 0 .0560 rpy=0 0 0; type static -> fixed
- joint claw: origin xyz=0 0 30.17 rpy=0 0 0 -> xyz=0 0 .03017 rpy=0 0 0; type static -> fixed
- joint elbow: limit lower=0 upper=1.0472 -> lower=0 upper=1.0472 effort=1000.0 velocity=0.5; origin xyz=0 0 118.65 rpy=0 0 0 -> xyz=0 0 .11865 rpy=0 1.57 0
- joint shoulder: limit lower=0.261799 upper=3.14 -> lower=0 upper=2.87979 effort=1000.0 velocity=0.5; origin xyz=0 0 120.0 rpy=0 0 0 -> xyz=0 0 0 rpy=0 0 0
- joint waist: limit lower=-1.57 upper=1.57 -> lower=-1.57 upper=1.57 effort=1000.0 velocity=0.5; origin xyz=0 0 42.93 rpy=0 0 1.57 -> xyz=0 0 .04293 rpy=0 0 1.57
- joint wrist_pitch: limit lower=0 upper=3.14 -> lower=0 upper=3.14 effort=1000.0 velocity=0.5; origin xyz=0 0 30.17 rpy=0 0 0 -> xyz=0 0 .03017 rpy=0 -1.309 0
- joint wrist_roll: limit lower=0 upper=3.14 -> lower=0 upper=3.14 effort=1000.0 velocity=0.5; origin xyz=0 0 60.028 rpy=0 0 0 -> xyz=0 0 .060028 rpy=0 0 1.57
