Commit message: pykdl w/ urdf attempt

File: arm_controller/urdf/ex.urdf (robot description, URDF)
Before this commit: robot example_robot, 4 links, 3 joints
Links:
- link link1: geometry visual box size=0.1 0.2 1
- link link2: geometry visual box size=0.1 0.5 .1; visual box size=0.5 0.1 .1
- link link3: geometry visual box size=1 .1 0.1
- link link4: geometry visual box size=1 0.1 0.1
Joints:
- joint joint1_2: origin xyz=5 3 0 rpy=0 0 0 -> xyz=0 0 1 rpy=0 0 0
- joint joint2_3: origin xyz=-2 5 0 rpy=0 0 1.57 -> xyz=-.5 .5 0 rpy=0 0 1.57
- joint joint3_4: origin xyz=5 0 0 rpy=0 0 -1.57 -> xyz=1 0 0 rpy=0 0 -1.57

Commit message: merged URDF, finished main urdf stuff, standardized all current solver returns

File: arm_controller/urdf/ex.urdf (robot description, URDF)
Before this commit: robot example_robot, 4 links, 3 joints
Links:
- added link link0; visual box size=1 0.1 0.1
Joints:
- added joint joint0_1: type fixed, parent link0, child link1, origin xyz=0 0 0 rpy=0 0 0

Commit message: comment style standardized, urdf fleshed out and given None assignments where needed

File: arm_controller/urdf/ex.urdf (robot description, URDF)
Before this commit: robot example_robot, 5 links, 4 joints
Links:
- link link0: geometry visual box size=0.3 0.3 0.3
- link link1: geometry visual cylinder length=1 radius=.1
Joints:
- joint joint0_1: axis (none) -> 0 0 1
- joint joint1_2: limit (none) -> effort=1000.0 velocity=0.5

Commit message: URDF limit adaptation

File: arm_controller/urdf/ex.urdf (robot description, URDF)
Before this commit: robot example_robot, 5 links, 4 joints
Joints:
- joint joint0_1: type fixed -> continuous
- joint joint1_2: limit effort=1000.0 velocity=0.5 -> lower=-1.57 upper=3.14 effort=1000.0 velocity=0.5; type continuous -> revolute
- joint joint2_3: limit (none) -> effort=1000.0 velocity=0.5
- joint joint3_4: axis 0.707 -0.707 0 -> (none); limit (none) -> lower=-1 upper=0 effort=1000.0 velocity=0.5; type continuous -> prismatic
