Commit message: updates

File: arm_controller/urdf/mechatronics_arm.urdf (robot description, URDF)
Before this commit: robot MechaArm, 10 links, 9 joints
Links:
- link claw_left_link: geometry visual box size=0.012 0.02 0.06
- link claw_right_link: geometry visual box size=0.012 0.02 0.06
- link elbow_wrist_roll_link: geometry visual box size=0.030 0.015 0.06; visual cylinder length=0.02 radius=0.015
- link shoulder_elbow_link: geometry visual box size=0.030 0.015 0.120; visual cylinder length=0.02 radius=0.015
- link waist_shoulder_link: geometry visual box size=0.030 0.015 0.042; visual cylinder length=0.02 radius=0.015
- link wrist_pitch_claw_link: geometry visual box size=0.012 0.03 0.03
- link wrist_roll_wrist_pitch_link: geometry visual box size=0.024 0.012 0.03; visual cylinder length=0.015 radius=0.01

Commit message: changes to plotter and surrounding classes to get plotter to plot w/ urdf

File: arm_controller/urdf/mechatronics_arm.urdf (robot description, URDF)
Before this commit: robot Mechatronics Arm, 10 links, 9 joints
Links:
- removed link claw_left_link
- removed link claw_right_link
Joints:
- removed joint claw_left
- removed joint claw_right

Commit message: updated radians and limit testing

File: arm_controller/urdf/mechatronics_arm.urdf (robot description, URDF)
Before this commit: robot Mechatronics Arm, 8 links, 7 joints
Joints:
- joint shoulder: limit lower=0 upper=2.87979 effort=1000.0 velocity=0.5 -> lower=0.2618 upper=3.14 effort=1000.0 velocity=0.5
- joint waist: limit lower=-1.57 upper=1.57 effort=1000.0 velocity=0.5 -> lower=0 upper=3.14 effort=1000.0 velocity=0.5; origin xyz=0 0 .04293 rpy=0 0 1.57 -> xyz=0 0 .04293 rpy=0 0 0

Commit message: remove base link in urdf and working on fixing set joints

File: arm_controller/urdf/mechatronics_arm.urdf (robot description, URDF)
Before this commit: robot Mechatronics Arm, 8 links, 7 joints
Links:
- removed link world_base_link
Joints:
- removed joint base
- joint shoulder: origin xyz=0 0 0 rpy=0 2.87979 0 -> xyz=0 0 0 rpy=0 3.14 0

Commit message: fixed solution so it properly moves arm to correct position

File: arm_controller/urdf/mechatronics_arm.urdf (robot description, URDF)
Before this commit: robot Mechatronics Arm, 7 links, 6 joints
Joints:
- joint waist: origin xyz=0 0 .04293 rpy=0 0 0 -> xyz=0 0 0.09893 rpy=0 0 0
